Commit message: 完成

File: custom_envs/assets/m20_piper_single/M20_Piper_lightweight.urdf (robot description, URDF)
Before this commit: robot M20_Piper, 27 links, 26 joints
Links:
- link gripper_base: geometry collision box size=0.075 0.075 0.064; visual mesh filename=/home/mojie/taskdog/deps/deep_robotics_model/M20_Piper/urdf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
- link link7: geometry collision mesh filename=/home/mojie/taskdog/deps/deep_robotics_model/M20_Piper/urdf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; visual mesh filename=/home/mojie/taskdog/deps/deep_robotics_model/M20_Piper/urdf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
- link link8: geometry collision mesh filename=/home/mojie/taskdog/deps/deep_robotics_model/M20_Piper/urdf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; visual mesh filename=/home/mojie/taskdog/deps/deep_robotics_model/M20_Piper/urdf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
